File: SB_CAN_MAIN/SB_CAN_MAIN.kicad_sch (KiCad schematic)
At the start: 89 parts, among them J1 XT30PB_IN, J2 USB_C_Receptacle_USB2.0_16P, J3 Excluder, J4 PT100, J5 Hotend, J6 FAN2, J7 LDC, J8 FS, J9 FAN, Q1 BUK9M8R5-40EX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

Commit message: layout: add fan board
Parts:
- added C37: 47pF, Capacitor_SMD:C_0402_1005Metric, symbol Device:C_Small
- added TP1, TP2: PAD, Library:PAD, symbol Connector:TestPoint_Small
- H1, H2: value MountingHole_Pad -> M3; footprint MountingHole:MountingHole_3.2mm_M3_DIN965_Pad -> MountingHole:MountingHole_3.2mm_M3_ISO14580_Pad
Connections:
- net +24V: now also TP1.1
- net +5V: now also C37.2
- net at D2.1 (K), J5.2 (Pin_2), Q1.5 (D): now also TP2.1
- net at R12.1, R13.1, U4.4 (VFB): now also C37.1
Other:
- moved on the sheet: H1, H2

Commit message: sch: fix bug that the tja1044 can only use 5V power
Connections:
- net +3V3A: no longer C14.1, U3.3 (VCC)
- net +5V: now also C14.1, U3.3 (VCC)
Changed lines of the file:
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@@
-	)
-	(symbol
-		(lib_id "power:+3V3")
-		(at 109.22 198.12 0)
-		(unit 1)
-		(exclude_from_sim no)
-		(in_bom yes)
-		(on_board yes)
-		(dnp no)
-		(fields_autoplaced yes)
-		(property "Reference" "#PWR0119"
-			(at 109.22 201.93 0)
-			(effects
-				(font
-					(size 1.27 1.27)
-				)
-				(hide yes)
-			)
-		)
-		(property "Value" "+3V3A"
-			(at 109.22 193.04 0)
-			(effects
-				(font
-					(size 1.27 1.27)
-				)
-			)
-		)
-		(property "Footprint" ""
-			(at 109.22 198.12 0)
-			(effects
-				(font
-					(size 1.27 1.27)
-				)
-				(hide yes)
-			)
-		)
-		(property "Datasheet" ""
-			(at 109.22 198.12 0)
-			(effects
-				(font
-					(size 1.27 1.27)
-				)
-				(hide yes)
-			)
-		)
-		(property "Description" "Power symbol creates a global label with name \"+3V3\""
-			(at 109.22 198.12 0)
-			(effects
-				(font
-					(size 1.27 1.27)
-				)
-				(hide yes)
-			)
-		)
-		(pin "1"
-		)
-		(instances
-			(project "SB_CAN_MAIN"
-				(path "/e3d9bf3f-f8be-4a0d-9b69-f1016d65a8ba"
-					(reference "#PWR0119")
-					(unit 1)
-				)
-			)
-		)
 	)
 	(symbol
@@
 					(unit 1)
 				)
+			)
+		)
+	)
+	(symbol
+		(lib_id "power:+5V")
+		(at 109.22 198.12 0)
+		(unit 1)
+		(exclude_from_sim no)
+		(in_bom yes)
+		(on_board yes)
+		(dnp no)
+		(fields_autoplaced yes)
+		(property "Reference" "#PWR017"
+			(at 109.22 201.93 0)
+			(effects
+				(font
+					(size 1.27 1.27)
+				)
+				(hide yes)
+			)
+		)
+		(property "Value" "+5V"
+			(at 109.22 193.04 0)
+			(effects
+				(font
+					(size 1.27 1.27)
+				)
+			)
+		)
+		(property "Footprint" ""
+			(at 109.22 198.12 0)
+			(effects
+				(font
+					(size 1.27 1.27)
+				)
+				(hide yes)
+			)
+		)
+		(property "Datasheet" ""
+			(at 109.22 198.12 0)
+			(effects
+				(font
+					(size 1.27 1.27)
+				)
+				(hide yes)
+			)
+		)
+		(property "Description" "Power symbol creates a global label with name \"+5V\""
+			(at 109.22 198.12 0)
+			(effects
+				(font
+					(size 1.27 1.27)
+				)
+				(hide yes)
+			)
+		)
+		(pin "1"
+		)
+		(instances
+			(project "SB_CAN_MAIN"
+				(path "/e3d9bf3f-f8be-4a0d-9b69-f1016d65a8ba"
+					(reference "#PWR017")
+					(unit 1)
+				)
