File: SB-fan-board/SB-fan-board.kicad_sch (KiCad schematic)
At the start: 15 parts, among them J1 FAN0, J2 FAN1, J3 NEO, J4 MAIN, U1 TPS54302

Commit message: generate gerber files
Connections:
- net ADC0: no longer names the net of J4.5 (Pin_5)
- net ADC1: no longer names the net of J4.7 (Pin_7)
- no-connect marks 0 -> 2
Changed lines of the file:
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@@
 		(color 0 0 0 0)
 	)
+	(no_connect
+		(at 69.85 93.98)
+	)
+	(no_connect
+		(at 69.85 96.52)
+	)
 	(wire
 		(pts
@@
 	(wire
 		(pts
-			(xy 69.85 96.52) (xy 59.69 96.52)
-		)
-		(stroke
-			(width 0)
-			(type default)
-		)
-	)
-	(wire
-		(pts
 			(xy 83.82 116.84) (xy 83.82 114.3)
 		)
@@
 	(wire
 		(pts
-			(xy 59.69 93.98) (xy 69.85 93.98)
-		)
-		(stroke
-			(width 0)
-			(type default)
-		)
-	)
-	(wire
-		(pts
 			(xy 86.36 123.19) (xy 83.82 123.19)
 		)
@@
 		)
 	)
-	(label "ADC0"
-		(at 59.69 93.98 0)
+	(label "FAN1_PWM"
+		(at 92.71 91.44 180)
 		(fields_autoplaced yes)
 		(effects
@@
 				(size 1.27 1.27)
 			)
-			(justify left bottom)
-		)
-	)
-	(label "FAN1_PWM"
-		(at 92.71 91.44 180)
+			(justify right bottom)
+		)
+	)
+	(label "FAN1_DET"
+		(at 113.03 100.33 0)
 		(fields_autoplaced yes)
 		(effects
@@
 				(size 1.27 1.27)
 			)
-			(justify right bottom)
-		)
-	)
-	(label "FAN1_DET"
-		(at 113.03 100.33 0)
+			(justify left bottom)
+		)
+	)
+	(label "FAN0_PWM"
+		(at 113.03 88.9 0)
 		(fields_autoplaced yes)
 		(effects
@@
 	)
 	(label "FAN0_PWM"
-		(at 113.03 88.9 0)
+		(at 59.69 91.44 0)
 		(fields_autoplaced yes)
 		(effects
@@
 		)
 	)
-	(label "FAN0_PWM"
-		(at 59.69 91.44 0)
+	(label "NEO"
+		(at 92.71 88.9 180)
 		(fields_autoplaced yes)
 		(effects
@@
 				(size 1.27 1.27)
 			)
-			(justify left bottom)
-		)
-	)
-	(label "NEO"
-		(at 92.71 88.9 180)
+			(justify right bottom)
+		)
+	)
+	(label "FAN1_PWM"
+		(at 113.03 102.87 0)
 		(fields_autoplaced yes)
 		(effects
@@
 				(size 1.27 1.27)
 			)
-			(justify right bottom)
-		)
-	)
-	(label "FAN1_PWM"
-		(at 113.03 102.87 0)
+			(justify left bottom)
+		)
+	)
+	(label "FAN1_DET"
+		(at 92.71 93.98 180)
 		(fields_autoplaced yes)
 		(effects
@@
 				(size 1.27 1.27)
 			)
-			(justify left bottom)
-		)
-	)
-	(label "FAN1_DET"
-		(at 92.71 93.98 180)
+			(justify right bottom)
+		)
+	)
+	(label "FAN0_DET"
+		(at 113.03 86.36 0)
 		(fields_autoplaced yes)
 		(effects
@@
 				(size 1.27 1.27)
 			)
-			(justify right bottom)
-		)
-	)
-	(label "FAN0_DET"
-		(at 113.03 86.36 0)
+			(justify left bottom)
+		)
+	)
+	(label "NEO"
+		(at 113.03 114.3 0)
 		(fields_autoplaced yes)
 		(effects
@@
 		)
 	)
-	(label "NEO"
-		(at 113.03 114.3 0)
+	(label "FAN0_DET"
+		(at 59.69 88.9 0)
 		(fields_autoplaced yes)
 		(effects
@@
 		)
 	)
-	(label "FAN0_DET"
-		(at 59.69 88.9 0)
-		(fields_autoplaced yes)
-		(effects
-			(font
-				(size 1.27 1.27)
-			)
-			(justify left bottom)
-		)
-	)
-	(label "ADC1"
-		(at 59.69 96.52 0)
-		(fields_autoplaced yes)
-		(effects
-			(font
-				(size 1.27 1.27)
-			)
-			(justify left bottom)
-		)
-	)
 	(symbol
 		(lib_id "Mechanical:MountingHole_Pad")
@@
 		)
 		(instances
-			(project "SB_CAN_FAN"
+			(project "SB-fan-board"
 				(path "/75679a6a-89de-45d6-8f1f-aa62e92337b9"
 					(reference "H2")
@@
 		)
 		(instances
-			(project "SB_CAN_FAN"
+			(project "SB-fan-board"
 				(path "/75679a6a-89de-45d6-8f1f-aa62e92337b9"
 					(reference "#PWR012")
@@
 		)
 		(instances
-			(project "SB_CAN_FAN"
+			(project "SB-fan-board"
 				(path "/75679a6a-89de-45d6-8f1f-aa62e92337b9"
 					(reference "#PWR014")
@@
 		)
 		(instances
-			(project "SB_CAN_FAN"
+			(project "SB-fan-board"
 				(path "/75679a6a-89de-45d6-8f1f-aa62e92337b9"
 					(reference "C3")
@@
 		)
 		(instances
-			(project "SB_CAN_FAN"
+			(project "SB-fan-board"
 				(path "/75679a6a-89de-45d6-8f1f-aa62e92337b9"
 					(reference "#PWR09")
@@
 		)
 		(instances
-			(project "SB_CAN_FAN"
+			(project "SB-fan-board"
 				(path "/75679a6a-89de-45d6-8f1f-aa62e92337b9"
 					(reference "C1")
@@
 		)
 		(instances
-			(project "SB_CAN_FAN"
+			(project "SB-fan-board"
 				(path "/75679a6a-89de-45d6-8f1f-aa62e92337b9"
 					(reference "H1")
@@
 		)
 		(instances
-			(project "SB_CAN_FAN"
+			(project "SB-fan-board"
 				(path "/75679a6a-89de-45d6-8f1f-aa62e92337b9"
 					(reference "#PWR06")
@@
 		)
 		(instances
-			(project "SB_CAN_FAN"
+			(project "SB-fan-board"
 				(path "/75679a6a-89de-45d6-8f1f-aa62e92337b9"
 					(reference "#PWR05")
@@
 		)
 		(instances
-			(project "SB_CAN_FAN"
+			(project "SB-fan-board"
 				(path "/75679a6a-89de-45d6-8f1f-aa62e92337b9"
 					(reference "#PWR015")
@@
 		)
 		(instances
-			(project "SB_CAN_FAN"
+			(project "SB-fan-board"
 				(path "/75679a6a-89de-45d6-8f1f-aa62e92337b9"
 					(reference "#PWR07")
@@
 		)
 		(instances
-			(project "SB_CAN_FAN"
+			(project "SB-fan-board"
 				(path "/75679a6a-89de-45d6-8f1f-aa62e92337b9"
 					(reference "R2")
@@
 		)
 		(instances
-			(project "SB_CAN_FAN"
+			(project "SB-fan-board"
 				(path "/75679a6a-89de-45d6-8f1f-aa62e92337b9"
 					(reference "J1")
@@
 		)
 		(instances
-			(project "SB_CAN_FAN"
+			(project "SB-fan-board"
 				(path "/75679a6a-89de-45d6-8f1f-aa62e92337b9"
 					(reference "#PWR011")
@@
 		)
 		(instances
-			(project "SB_CAN_FAN"
+			(project "SB-fan-board"
 				(path "/75679a6a-89de-45d6-8f1f-aa62e92337b9"
 					(reference "C2")
@@
 		)
 		(instances
-			(project "SB_CAN_FAN"
+			(project "SB-fan-board"
 				(path "/75679a6a-89de-45d6-8f1f-aa62e92337b9"
 					(reference "R3")
@@
 		)
 		(instances
-			(project "SB_CAN_FAN"
+			(project "SB-fan-board"
 				(path "/75679a6a-89de-45d6-8f1f-aa62e92337b9"
 					(reference "J2")
@@
 		)
 		(instances
-			(project "SB_CAN_FAN"
+			(project "SB-fan-board"
 				(path "/75679a6a-89de-45d6-8f1f-aa62e92337b9"
 					(reference "#PWR013")
@@
 		)
 		(instances
-			(project "SB_CAN_FAN"
+			(project "SB-fan-board"
 				(path "/75679a6a-89de-45d6-8f1f-aa62e92337b9"
 					(reference "#PWR010")
@@
 		)
 		(instances
-			(project "SB_CAN_FAN"
+			(project "SB-fan-board"
 				(path "/75679a6a-89de-45d6-8f1f-aa62e92337b9"
 					(reference "#PWR01")
@@
 		)
 		(instances
-			(project "SB_CAN_FAN"
+			(project "SB-fan-board"
 				(path "/75679a6a-89de-45d6-8f1f-aa62e92337b9"
 					(reference "#PWR04")
@@
 		)
 		(instances
-			(project "SB_CAN_FAN"
+			(project "SB-fan-board"
 				(path "/75679a6a-89de-45d6-8f1f-aa62e92337b9"
 					(reference "L1")
@@
 		)
 		(instances
-			(project "SB_CAN_FAN"
+			(project "SB-fan-board"
 				(path "/75679a6a-89de-45d6-8f1f-aa62e92337b9"
 					(reference "C4")
@@
 		)
 		(instances
-			(project "SB_CAN_FAN"
+			(project "SB-fan-board"
 				(path "/75679a6a-89de-45d6-8f1f-aa62e92337b9"
 					(reference "J4")
@@
 		)
 		(instances
-			(project "SB_CAN_FAN"
+			(project "SB-fan-board"
 				(path "/75679a6a-89de-45d6-8f1f-aa62e92337b9"
 					(reference "#PWR02")
@@
 		)
 		(instances
-			(project "SB_CAN_FAN"
+			(project "SB-fan-board"
 				(path "/75679a6a-89de-45d6-8f1f-aa62e92337b9"
 					(reference "#PWR08")
@@
 		)
 		(instances
-			(project "SB_CAN_FAN"
+			(project "SB-fan-board"
 				(path "/75679a6a-89de-45d6-8f1f-aa62e92337b9"
 					(reference "J3")
@@
 		)
 		(instances
-			(project "SB_CAN_FAN"
+			(project "SB-fan-board"
 				(path "/75679a6a-89de-45d6-8f1f-aa62e92337b9"
 					(reference "U1")
@@
 		)
 		(instances
-			(project "SB_CAN_FAN"
+			(project "SB-fan-board"
 				(path "/75679a6a-89de-45d6-8f1f-aa62e92337b9"
 					(reference "#PWR03")
@@
 		)
 		(instances
-			(project "SB_CAN_FAN"
+			(project "SB-fan-board"
 				(path "/75679a6a-89de-45d6-8f1f-aa62e92337b9"
 					(reference "R1")
