File: SB-main-board/SB-main-board.kicad_pcb (KiCad board)
At the start: 4 copper layers, 53 x 40 mm, 95 parts, among them J1 XT30PB_IN, J2 USB_C_Receptacle_USB2.0_16P, J3 Excluder, J4 PT100, J5 Hotend, J6 FAN2, J7 LDC, J8 FS, J9 FAN, Q1 BUK9M8R5-40EX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

Commit message: silkscreen: add more information
Parts:
- added REF**: OSHW-Logo2_7.3x6mm_SilkScreen, Symbol:OSHW-Logo2_7.3x6mm_SilkScreen, B.Cu at (77.4, 71.8)
- added REF**: KiCad-Logo2_6mm_SilkScreen, Symbol:KiCad-Logo2_6mm_SilkScreen, B.Cu at (92.5, 70.9)
- moved FB4 48.3 mm to (97.3, 84.1)
- moved C10 48.3 mm to (122.2, 96.8)
- moved C13 48.3 mm to (115.9, 94.3)
- moved C21 48.3 mm to (114.1, 77.0)
- moved C27 48.3 mm to (111.9, 70.5)
- moved C28 48.3 mm to (108.8, 70.5)
- moved C3 48.3 mm to (124.0, 106.4)
- moved C30 48.3 mm to (77.4, 90.7)
- moved C6 48.3 mm to (115.2, 95.0)
- moved C8 48.3 mm to (121.6, 103.2)
- moved D1 48.3 mm to (124.7, 101.7)
- moved D2 48.3 mm to (102.7, 82.8)
- moved D3 48.3 mm to (115.7, 88.0)
- moved FB2 48.3 mm to (124.0, 78.2)
- moved H1 48.3 mm to (98.1, 80.1)
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Other:
- board text added: "0"
- board text added: "0 mm"
- board text added: "0.01 mm"
- board text added: "0.02"
- board text added: "0.035 mm"
- board text added: "0.0889 mm / 0.0889 mm"
- board text added: "0.1 mm"
- board text added: "0.3000 mm"
- board text added: "1"
- board text added: "1.24 mm"
- board text added: "1.6000 mm"
- board text added: "3.3"
- board text added: "4"
- board text added: "4.5"
- board text added: "4W"
- board text added: "53.0000 mm x 40.0000 mm"
- board text added: "B.Cu"
- board text added: "B.Mask"
- board text added: "B.Paste"
- board text added: "B.Silkscreen"
- board text added: "BOARD CHARACTERISTICS"
- board text added: "Bottom Silk Screen"
- board text added: "Bottom Solder Mask"
- board text added: "Bottom Solder Paste"
- board text added: "Direct Printing"
- board text added: "Epsilon R"
- board text added: "F.Cu"
- board text added: "F.Mask"
- board text added: "F.Paste"
- board text added: "F.Silkscreen"
- board text added: "FR4"
- board text added: "FR4 natural"
- board text added: "Green"
- board text added: "Immersion gold"
- board text added: "In1.Cu"
- board text added: "In2.Cu"
- board text added: "Liquid Ink"
- board text added: "Loss Tangent"
- board text added: "REF"
- board text added: "STEP"
- board text added: "Terminal Resistor"
- board text added: "Top Silk Screen"
- board text added: "Top Solder Mask"
- board text added: "Top Solder Paste"
- board text added: "White"
- board text added: "copper"
- board text added: "core"
- board text added: "prepreg"
- board text added: "介质 1"
- board text added: "介质 2"
- board text added: "介质 3"
- board text added: "厚度 (mm)"
- board text added: "否"
- board text added: "存在半孔焊盘:"
- board text added: "层名称"
- board text added: "最小孔径:"
- board text added: "最小走线/间距:"
- board text added: "材料"
- board text added: "板厚:"
- board text added: "板子整体尺寸:"
- board text added: "板边倒角处理:"
- board text added: "类型"
- board text added: "铜层数量:"
- board text added: "镀铜处理:"
- board text added: "阻抗控制:"
- board text added: "需要电镀板边:"
- board text added: "颜色"

Commit message: sch: optimize return path
Parts:
- added FB5: 120R@100MHz, Inductor_SMD:L_0603_1608Metric, B.Cu at (97.3, 84.1)
- FB4: moved to F.Cu
- moved FB4 9.71 mm to (93.2, 75.3), turned to -90 degrees
Connections:
- FB4 pad 1: +3V3B -> GND
- FB4 pad 2: Net-(U9-VDD) -> PGND
Routing:
- net PGND: vias 41 -> 42
