File: SB-main-board/SB-main-board.kicad_sch (KiCad schematic)
At the start: 89 parts, among them J1 XT30PB_IN, J2 Download, J3 Excluder, J4 PT100, J5 Hotend, J6 FAN2, J7 LDC, J8 FS, J9 FAN, Q1 BUK9M4R3-40H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

Commit message: misc: fix typo
Parts:
- R16: value 220mR -> 200mR
Changed lines of the file:
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@@
 			)
 		)
-		(property "Value" "220mR"
+		(property "Value" "200mR"
 			(at 224.79 93.98 0)
 			(effects

Commit message: misc: update all files to kicad 9
Parts:
- U6: symbol Library:TMC2208-LA -> Library:TMC2209-LA
Changed lines of the file:
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@@
 			)
 		)
+		(property "Sim.Pins" "1=K 2=A"
+			(at 49.53 144.78 0)
+			(effects
+				(font
+					(size 1.27 1.27)
+				)
+				(hide yes)
+			)
+		)
 		(pin "2"
 		)
@@
 	)
 	(symbol
-		(lib_id "Library:TMC2208-LA")
+		(lib_id "Library:TMC2209-LA")
 		(at 189.23 67.31 0)
 		(unit 1)
@@
 			)
 		)
+		(property "Sim.Pins" "1=K 2=A"
+			(at 267.97 24.13 0)
+			(effects
+				(font
+					(size 1.27 1.27)
+				)
+				(hide yes)
+			)
+		)
 		(pin "2"
 		)
@@
 			)
 		)
-		(property "Description" ""
+		(property "Description" "Power symbol creates a global label with name \"GND\" , ground"
 			(at 59.69 241.3 0)
 			(effects
